File: PCB-source/CAN_TR.kicad_sch (KiCad schematic)
At the start: 4 parts, among them U500 TJA1044GTK_3Z

Commit message: bom done
Parts:
- U500: LCSC (none) -> C5215851
Changed lines of the file:
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@@
+			)
+		)
+		(property "LCSC" "C5215851"
+			(at 128.27 92.71 0)
+			(effects
+				(font
+					(size 1.27 1.27)
+				)
+				(hide yes)
 			)
 		)
