File: PCB-source/LMR36520ADDAR.kicad_sch (KiCad schematic)
At the start: 32 parts, among them U2 LMR36520ADDAR

Commit message: DRC PASS, preparing bom for production
Parts:
- removed D402: Red, PCM_JLCPCB:D_0603, symbol PCM_JLCPCB-Diodes:LED,0603,Red
- removed R12: 1.2kΩ, PCM_JLCPCB:R_0402, symbol PCM_JLCPCB-Resistors:0402,1.2kΩ
- removed R6: 100kΩ, PCM_JLCPCB:R_0402, symbol PCM_JLCPCB-Resistors:0402,100kΩ
- added R12: 100kΩ, PCM_JLCPCB:R_0603, symbol PCM_JLCPCB-Resistors:0603,100kΩ
Connections:
- net FB: now also R12.2
- net Vout: now also R12.1

Commit message: bom done
Parts:
- L1: LCSC (none) -> C917354
- U2: LCSC (none) -> C2879422
Other:
- note added: "NO ALTERNATE PART AVALIABLE IF F-version is choosen instead of A-version it will have lower efficency at lower current due to F-ver being fixed freq"
- note added: "NOTE:"
Changed lines of the file:
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@@
 	)
 	(rectangle
+		(start 71.12 129.54)
+		(end 118.11 142.24)
+		(stroke
+			(width 0)
+			(type default)
+		)
+		(fill
+			(type none)
+		)
+	)
+	(rectangle
+		(start 71.12 124.46)
+		(end 118.11 129.54)
+		(stroke
+			(width 0)
+			(type default)
+		)
+		(fill
+			(type none)
+		)
+	)
+	(rectangle
 		(start 30.48 34.036)
 		(end 148.59 39.116)
@@
 		)
 	)
+	(text "NO ALTERNATE PART AVALIABLE\nIF F-version is choosen instead of A-version\nit will have lower efficency at lower current \ndue to F-ver being fixed freq"
+		(exclude_from_sim no)
+		(at 71.882 135.89 0)
+		(effects
+			(font
+				(size 1.27 1.27)
+				(thickness 0.254)
+				(bold yes)
+				(color 255 45 78 1)
+			)
+			(justify left)
+		)
+	)
+	(text "NOTE:"
+		(exclude_from_sim no)
+		(at 71.628 127.254 0)
+		(effects
+			(font
+				(size 2.54 2.54)
+				(thickness 0.254)
+				(bold yes)
+			)
+			(justify left)
+		)
+	)
 	(text "INFORMATION"
 		(exclude_from_sim no)
@@
 			)
 		)
+		(property "LCSC" "C917354"
+			(at 162.56 80.01 90)
+			(effects
+				(font
+					(size 1.27 1.27)
+				)
+				(hide yes)
+			)
+		)
 		(pin "1"
 		)
@@
 			(at 128.27 82.55 0)
 			(effects
+				(font
+					(size 1.27 1.27)
+				)
+				(hide yes)
+			)
+		)
+		(property "LCSC" "C2879422"
+			(at 128.27 82.55 0)
+			(effects
