File: PCB-source/LMR74700.kicad_sch (KiCad schematic)
At the start: 4 parts, among them Q7 AO3400A, U5 LM74700

Commit message: bom done
Parts:
- U5: LCSC (none) -> C2941042
Other:
- note added: "ALTERNATE PART: Wuxi Maxinmicro MX74700T PIN COMPATIBLE."
- note added: "NOTE:"
- moved on the sheet: Q7
