File: PCB-source/POWER_CONN.kicad_sch (KiCad schematic)
At the start: 1 part, among them J7 AMASS XT60

Commit message: bom done
Parts:
- J7: LCSC (none) -> C428722
Changed lines of the file:
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@@
+			)
+		)
+		(property "LCSC" "C428722"
+			(at 128.27 97.79 0)
+			(effects
+				(font
+					(size 1.27 1.27)
+				)
+				(hide yes)
 			)
 		)
