File: PCB-source/POWER_IN_CONN.kicad_sch (KiCad schematic)
At the start: 1 part, among them J2 AMASS XT60

Commit message: bom done
Parts:
- J2: LCSC (none) -> C98732
Changed lines of the file:
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@@
+			)
+		)
+		(property "LCSC" "C98732"
+			(at 134.62 100.33 0)
+			(effects
+				(font
+					(size 1.27 1.27)
+				)
+				(hide yes)
 			)
 		)
