File: PCB-source/USB HUB.kicad_sch (KiCad schematic)
At the start: 15 parts, among them U302 CH334P, Y900 Crystal_GND24

Commit message: bom done
Parts:
- Y900: LCSC (none) -> C9002
Changed lines of the file:
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@@
+			)
+		)
+		(property "LCSC" "C9002"
+			(at 187.96 90.17 90)
+			(effects
+				(font
+					(size 1.27 1.27)
+				)
+				(hide yes)
 			)
 		)
