File: PCB-source/USB switch.kicad_sch (KiCad schematic)
At the start: 5 parts, among them U801 FSUSB42UMX

Commit message: bom done
Parts:
- U801: LCSC (none) -> C11145
Other:
- note added: "ALTERNATE PART: EnergyMath EMS3900 1.9Ω 800MHz 2:1 USB QFN-10L(1.4x1.8) Analog Switches - Special Purpose ROHS PIN COMPATIBLE"
- note added: "NOTE:"
Changed lines of the file:
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@@
 		(comment 2 "Designed in poland")
+	)
+	(rectangle
+		(start 171.45 110.49)
+		(end 215.9 115.57)
+		(stroke
+			(width 0)
+			(type default)
+		)
+		(fill
+			(type none)
+		)
+	)
+	(rectangle
+		(start 171.45 115.57)
+		(end 215.9 128.27)
+		(stroke
+			(width 0)
+			(type default)
+		)
+		(fill
+			(type none)
+		)
+	)
+	(text "NOTE:"
+		(exclude_from_sim no)
+		(at 171.958 113.284 0)
+		(effects
+			(font
+				(size 2.54 2.54)
+				(thickness 0.254)
+				(bold yes)
+			)
+			(justify left)
+		)
+	)
+	(text "ALTERNATE PART:\nEnergyMath EMS3900\n1.9Ω 800MHz 2:1 USB QFN-10L(1.4x1.8) \nAnalog Switches - Special Purpose ROHS\nPIN COMPATIBLE"
+		(exclude_from_sim no)
+		(at 172.212 121.92 0)
+		(effects
+			(font
+				(size 1.27 1.27)
+				(thickness 0.254)
+				(bold yes)
+				(color 255 45 78 1)
+			)
+			(justify left)
+		)
 	)
 	(junction
@@
 				(hide yes)
 			)
+		)
+		(property "LCSC" "C11145"
+			(at 137.16 88.9 0)
+			(effects
+				(font
+					(size 1.27 1.27)
+				)
+				(hide yes)
+			)
