File: PCB-source/USBC_CONN.kicad_sch (KiCad schematic)
At the start: 7 parts, among them J800 USB_C_Receptacle_USB2.0_16P, U401 TPD2EUSB30DRTR-TP

Commit message: bom done
Parts:
- J800: LCSC (none) -> C165948
Changed lines of the file:
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@@
+			)
+		)
+		(property "LCSC" "C165948"
+			(at 101.6 87.63 0)
+			(effects
+				(font
+					(size 1.27 1.27)
+				)
+				(hide yes)
 			)
 		)
