File: PCB-source/MMS2.kicad_pcb (KiCad board)
At the start: 4 copper layers, 90 x 50 mm, 192 parts, among them J1 86093488324755V1LF, J2 AMASS XT60, J3 Programming header, J4 Conn_01x16_Socket, J5 Conn_01x03_Pin, J7 AMASS XT60, J8 RJ45_LED_Shielded, J800 USB_C_Receptacle_USB2.0_16P, J9 RJ45_LED_Shielded, Q7 AO3400A, Q700 MMST3904, SW1 BOOT, SW2 RESET, U1 STM32F405RGTx, U2 LMR36520ADDAR, U3 TPD2EUSB30DRTR-TP, U301 TPS563200, U302 CH334P, U4 TPD2EUSB30DRTR-TP, U401 TPD2EUSB30DRTR-TP, U5 LM74700, U500 TJA1044GTK_3Z, U501 TJA1044GTK_3Z, U6 AT24C256C, U7 CH32V003FxUx, U700 STM32F103CBTx, U8 TLP175A, U801 FSUSB42UMX, U9 TLP175A, X1 X32258MOB4SI, X2 Q13FC1350000400, Y700 Crystal_GND24, Y900 Crystal_GND24

Commit message: bom done
Parts:
- removed C46: 10n, Capacitor_SMD:C_0402_1005Metric
- removed R55: 1k, Resistor_SMD:R_0402_1005Metric
- removed R56: 33k, Resistor_SMD:R_0402_1005Metric
- added C34: 10nF, PCM_JLCPCB:C_0402, F.Cu at (154.6, 103.4)
- added R27: 33kΩ, PCM_JLCPCB:R_0402, F.Cu at (154.6, 104.3)
- added R6: 1kΩ, PCM_JLCPCB:R_0402, F.Cu at (155.1, 120.2)
- C45: value 10n -> 10nF; footprint Capacitor_SMD:C_0402_1005Metric -> PCM_JLCPCB:C_0402
- R51: value 33k -> 33kΩ; footprint Resistor_SMD:R_0402_1005Metric -> PCM_JLCPCB:R_0402
- R53: value 1k -> 1kΩ; footprint Resistor_SMD:R_0402_1005Metric -> PCM_JLCPCB:R_0402
- R712: value 1.2kΩ -> 1.5kΩ
- moved D4 0.40 mm to (115.3, 114.4)
- moved NT2 0.33 mm to (104.1, 131.3)
- moved D3 0.30 mm to (115.3, 119.6)
- turned R53 to -90 degrees
Connections:
- R53 pad 1: /MCU/USER_LED_1 -> Net-(J8-Pad12)
- R53 pad 2: Net-(J8-Pad12) -> /MCU/USER_LED_1
Routing:
- net GND: track 118.8 -> 120.4 mm, vias 187 -> 191
- net +3V3: track 105.1 -> 103.8 mm
- net /CAN_TR1/CAN.RX: track 46.3 -> 47.1 mm

Commit message: REV A production ready
Parts:
- added ?: , , F.Cu at (84.0, 135.0)
- added ?: , , F.Cu at (167.0, 135.0)
- added G***: LOGO, QRcode:QR, B.Cu at (106.2, 117.5)
- added REF**: ESD-Logo_6.6x6mm_SilkScreen, Symbol:ESD-Logo_6.6x6mm_SilkScreen, F.Cu at (103.5, 122.7)
- added REF**: Hole_Tooling_JLCPCB, PCM_JLCPCB:Hole_Tooling_JLCPCB, F.Cu at (167.0, 90.0)
- added REF**: ESD-Logo_8.9x8mm_SilkScreen, Symbol:ESD-Logo_8.9x8mm_SilkScreen, B.Cu at (101.0, 103.5)
- added REF**: Part_Num_JLCPCB, PCM_JLCPCB:Part_Num_JLCPCB, B.Cu at (149.2, 112.5)
- added REF**: WEEE-Logo_4.2x6mm_SilkScreen, Symbol:WEEE-Logo_4.2x6mm_SilkScreen, B.Cu at (108.2, 104.5)
- R13: value 680Ω -> 220Ω
- R53, R6: value 1kΩ -> 220Ω
- R707, R713: value 10kΩ -> 220Ω
- R711: value 39kΩ -> 24.9kΩ
Routing:
- net VBUS: track 40.0 -> 39.3 mm
- net GND: vias 191 -> 204
Other:
- board text added: "+"
- board text added: "-"
- board text added: "12V"
- board text added: "3V3"
- board text added: "5V0"
- board text added: "B G R C D 3"
- board text added: "C1+"
- board text added: "C1-"
- board text added: "C2+"
- board text added: "C2-"
- board text added: "DEVICE ESD SENSETIVE"
- board text added: "DM"
- board text added: "DP"
- board text added: "G"
- board text added: "GND"
- board text added: "IO R G"
- board text added: "N/C"
- board text added: "This is prototype device It is not certified according to current EU laws. Do not sell or use outside of research purposes."
- board text added: "i"
