File: PCB-source/STlink-BMprobe.kicad_sch (KiCad schematic)
At the start: 34 parts, among them J3 Programming header, Q700 MMST3904, U700 STM32F103CBTx, Y700 Crystal_GND24

Commit message: ch32
Parts:
- removed TP700, TP701: TestPoint, TestPoint:TestPoint_Pad_D1.0mm, symbol Connector:TestPoint
Connections:
- net STLINK_RX renamed STLINK.TX
- net STLINK_TX renamed STLINK.RX
Other:
- note added: "UART FLIP HERE"

Commit message: bom done
Parts:
- removed R712: 1.2kΩ, PCM_JLCPCB:R_0402, symbol PCM_JLCPCB-Resistors:0402,1.2kΩ
- added R712: 1.5kΩ, PCM_JLCPCB:R_0402, symbol PCM_JLCPCB-Resistors:0402,1.5kΩ
- J3: now left out of the parts list
- Q700: LCSC C22388837 -> C20526
- U700: LCSC (none) -> C8304
Connections:
- net ST-LINK.D+: now also R712.2
- net at Q700.2 (E): now also R712.1
Other:
- note added: "ALTERNATE PART: GigaDevice Semicon Beijing GD32F103CBT6 PIN AND FW COMPATIBLE WAZZUP BEIJING"
- note added: "NOTE:"

Commit message: REV A production ready
Parts:
- removed R707, R713: 10kΩ, PCM_JLCPCB:R_0402, symbol PCM_JLCPCB-Resistors:0402,10kΩ
- removed R711: 39kΩ, PCM_JLCPCB:R_0402, symbol PCM_JLCPCB-Resistors:0402,39kΩ
- added R707, R713: 220Ω, PCM_JLCPCB:R_0402, symbol PCM_JLCPCB-Resistors:0402,220Ω
- added R711: 24.9kΩ, PCM_JLCPCB:R_0402, symbol PCM_JLCPCB-Resistors:0402,24kΩ
Connections:
- net +3V3: now also R707.1
- net GND: now also R711.2, R713.2
- net at D701.1: now also R713.1
- net at Q700.1 (B), R709.2, R710.1: now also R711.1
- net at D700.2: now also R707.2
