File: PCB-source/TPS563200.kicad_sch (KiCad schematic)
At the start: 12 parts, among them U301 TPS563200

Commit message: Component placement done
Parts:
- removed TP302: TestPoint, TestPoint:TestPoint_Pad_D1.0mm, symbol Connector:TestPoint
Changed lines of the file:
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@@
-	)
-	(junction
-		(at 143.51 100.33)
-		(diameter 0)
-		(color 0 0 0 0)
 	)
 	(junction
@@
 	(wire
 		(pts
-			(xy 121.92 100.33) (xy 143.51 100.33)
-		)
-		(stroke
-			(width 0)
-			(type default)
-		)
-	)
-	(wire
-		(pts
-			(xy 143.51 100.33) (xy 151.13 100.33)
+			(xy 121.92 100.33) (xy 151.13 100.33)
 		)
 		(stroke
@@
 					(unit 1)
 				)
-			)
-		)
-	)
-	(symbol
-		(lib_id "Connector:TestPoint")
-		(at 143.51 100.33 0)
-		(unit 1)
-		(exclude_from_sim no)
-		(in_bom yes)
-		(on_board yes)
-		(dnp no)
-		(property "Reference" "TP302"
-			(at 143.51 95.25 0)
-			(effects
-				(font
-					(size 1.27 1.27)
-				)
-			)
-		)
-		(property "Value" "TestPoint"
-			(at 146.05 98.298 0)
-			(effects
-				(font
-					(size 1.27 1.27)
-				)
-				(justify left)
-				(hide yes)
-			)
-		)
-		(property "Footprint" "TestPoint:TestPoint_Pad_D1.0mm"
-			(at 148.59 100.33 0)
-			(effects
-				(font
-					(size 1.27 1.27)
-				)
-				(hide yes)
-			)
-		)
-		(property "Datasheet" "~"
-			(at 148.59 100.33 0)
-			(effects
-				(font
-					(size 1.27 1.27)
-				)
-				(hide yes)
-			)
-		)
-		(property "Description" "test point"
-			(at 143.51 100.33 0)
-			(effects
-				(font
-					(size 1.27 1.27)
-				)
-				(hide yes)
-			)
-		)
-		(pin "1"
-		)
-		(instances
-			(project "MMS2"
-				(path "/6596548a-44e0-46d8-8624-fd71cf4a3e17/c3406df1-7cb0-4484-a477-0c72b46ba076/d003e443-17a0-422c-b61a-990137afd07b"
-					(reference "TP302")
-					(unit 1)
-				)

Commit message: bom done
Parts:
- JP301: now left out of the parts list
- U301: LCSC (none) -> C116592
Other:
- note added: "NO ALTERNATE PART AVALIABLE Incompatible pinout. (tho at price of 0.2usd this is cheapest buck anyway)"
- note added: "NOTE:"
Changed lines of the file:
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@@
+	)
+	(rectangle
+		(start 69.85 128.27)
+		(end 125.73 133.35)
+		(stroke
+			(width 0)
+			(type default)
+		)
+		(fill
+			(type none)
+		)
+	)
+	(rectangle
+		(start 69.85 133.35)
+		(end 125.73 142.24)
+		(stroke
+			(width 0)
+			(type default)
+		)
+		(fill
+			(type none)
+		)
 	)
 	(rectangle
@@
 				(bold yes)
 			)
+		)
+	)
+	(text "NO ALTERNATE PART AVALIABLE\nIncompatible pinout.\n(tho at price of 0.2usd this is cheapest buck anyway)\n"
+		(exclude_from_sim no)
+		(at 70.612 138.176 0)
+		(effects
+			(font
+				(size 1.27 1.27)
+				(thickness 0.254)
+				(bold yes)
+				(color 255 45 78 1)
+			)
+			(justify left)
+		)
+	)
+	(text "NOTE:"
+		(exclude_from_sim no)
+		(at 70.358 131.064 0)
+		(effects
+			(font
+				(size 2.54 2.54)
+				(thickness 0.254)
+				(bold yes)
+			)
+			(justify left)
 		)
 	)
@@
 			)
 		)
+		(property "LCSC" "C116592"
+			(at 101.6 92.71 0)
+			(effects
+				(font
+					(size 1.27 1.27)
+				)
+				(hide yes)
+			)
+		)
 		(pin "5"
 		)
@@
 		(unit 1)
 		(exclude_from_sim no)
-		(in_bom yes)
+		(in_bom no)
 		(on_board yes)
 		(dnp no)

Commit message: REV A production ready
Parts:
- removed R13: 680Ω, PCM_JLCPCB:R_0402, symbol PCM_JLCPCB-Resistors:0402,680Ω
- added R13: 220Ω, PCM_JLCPCB:R_0402, symbol PCM_JLCPCB-Resistors:0402,220Ω
Connections:
- net GND: now also R13.2
- net at D2.1: now also R13.1
Changed lines of the file:
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@@
 	(wire
 		(pts
-			(xy 181.61 101.6) (xy 181.61 99.06)
+			(xy 181.61 99.06) (xy 181.61 101.6)
 		)
 		(stroke
@@
 	)
 	(symbol
-		(lib_id "PCM_JLCPCB-Resistors:0402,680Ω")
+		(lib_id "PCM_JLCPCB-Resistors:0402,220Ω")
 		(at 181.61 105.41 0)
 		(unit 1)
@@
 			)
 		)
-		(property "Value" "680Ω"
+		(property "Value" "220Ω"
 			(at 181.61 105.41 90)
 			(do_not_autoplace yes)
@@
 			)
 		)
-		(property "Datasheet" "https://www.lcsc.com/datasheet/lcsc_datasheet_2205311900_UNI-ROYAL-Uniroyal-Elec-0402WGF6800TCE_C25130.pdf"
+		(property "Datasheet" "https://www.lcsc.com/datasheet/lcsc_datasheet_2205311900_UNI-ROYAL-Uniroyal-Elec-0402WGF2200TCE_C25091.pdf"
 			(at 181.61 105.41 0)
 			(effects
@@
 			)
 		)
-		(property "Description" "62.5mW Thick Film Resistors 50V ±100ppm/°C ±1% 680Ω 0402 Chip Resistor - Surface Mount ROHS"
+		(property "Description" "62.5mW Thick Film Resistors 50V ±100ppm/°C ±1% 220Ω 0402 Chip Resistor - Surface Mount ROHS"
 			(at 181.61 105.41 0)
 			(effects
@@
 			)
 		)
-		(property "LCSC" "C25130"
+		(property "LCSC" "C25091"
 			(at 181.61 105.41 0)
 			(effects
@@
 			)
 		)
-		(property "Stock" "148945"
+		(property "Stock" "617243"
 			(at 181.61 105.41 0)
 			(effects
@@
 			)
 		)
-		(property "Class" "Preferred Component"
+		(property "Class" "Basic Component"
 			(at 181.61 105.41 0)
 			(effects
@@
 			)
 		)
-		(property "Part" "0402WGF6800TCE"
+		(property "Part" "0402WGF2200TCE"
 			(at 181.61 105.41 0)
 			(effects
@@
 			)
 		)
-		(property "Resistance" "680Ω"
+		(property "Resistance" "220Ω"
 			(at 181.61 105.41 0)
 			(effects
@@
 			)
 		)
+		(pin "1"
+		)
 		(pin "2"
 		)
-		(pin "1"
-		)
 		(instances
-			(project ""
+			(project "MMS2"
 				(path "/6596548a-44e0-46d8-8624-fd71cf4a3e17/c3406df1-7cb0-4484-a477-0c72b46ba076/d003e443-17a0-422c-b61a-990137afd07b"
 					(reference "R13")
