File: PCB-source/VRM.kicad_sch (KiCad schematic)
At the start: 0 parts

Commit message: DRC PASS, preparing bom for production
Changed lines of the file:
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@@
 	(wire
 		(pts
+			(xy 252.73 82.55) (xy 252.73 87.63)
+		)
+		(stroke
+			(width 0)
+			(type default)
+		)
+	)
+	(wire
+		(pts
 			(xy 181.61 87.63) (xy 191.77 87.63)
 		)
@@
 	(wire
 		(pts
-			(xy 166.37 130.81) (xy 181.61 130.81)
+			(xy 40.64 81.28) (xy 40.64 88.9)
 		)
 		(stroke
@@
 	(wire
 		(pts
-			(xy 166.37 124.46) (xy 166.37 130.81)
+			(xy 241.3 87.63) (xy 252.73 87.63)
 		)
 		(stroke
@@
 	(wire
 		(pts
-			(xy 40.64 81.28) (xy 40.64 88.9)
+			(xy 173.99 130.81) (xy 173.99 124.46)
 		)
 		(stroke
@@
 	(wire
 		(pts
+			(xy 181.61 130.81) (xy 173.99 130.81)
+		)
+		(stroke
+			(width 0)
+			(type default)
+		)
+	)
+	(wire
+		(pts
 			(xy 181.61 130.81) (xy 181.61 87.63)
 		)
@@
 	)
 	(symbol
+		(lib_id "power:+5V")
+		(at 173.99 124.46 0)
+		(unit 1)
+		(exclude_from_sim no)
+		(in_bom yes)
+		(on_board yes)
+		(dnp no)
+		(fields_autoplaced yes)
+		(property "Reference" "#PWR086"
+			(at 173.99 128.27 0)
+			(effects
+				(font
+					(size 1.27 1.27)
+				)
+				(hide yes)
+			)
+		)
+		(property "Value" "+5V"
+			(at 173.99 119.38 0)
+			(effects
+				(font
+					(size 1.27 1.27)
+				)
+			)
+		)
+		(property "Footprint" ""
+			(at 173.99 124.46 0)
+			(effects
+				(font
+					(size 1.27 1.27)
+				)
+				(hide yes)
+			)
+		)
+		(property "Datasheet" ""
+			(at 173.99 124.46 0)
+			(effects
+				(font
+					(size 1.27 1.27)
+				)
+				(hide yes)
+			)
+		)
+		(property "Description" "Power symbol creates a global label with name \"+5V\""
+			(at 173.99 124.46 0)
+			(effects
+				(font
+					(size 1.27 1.27)
+				)
+				(hide yes)
+			)
+		)
+		(pin "1"
+		)
+		(instances
+			(project ""
+				(path "/6596548a-44e0-46d8-8624-fd71cf4a3e17/c3406df1-7cb0-4484-a477-0c72b46ba076"
+					(reference "#PWR086")
+					(unit 1)
+				)
+			)
+		)
+	)
+	(symbol
 		(lib_id "power:VCC")
 		(at 40.64 81.28 0)
@@
 	)
 	(symbol
-		(lib_id "power:VBUS")
-		(at 166.37 124.46 0)
+		(lib_id "power:+3V3")
+		(at 252.73 82.55 0)
 		(unit 1)
 		(exclude_from_sim no)
@@
 		(fields_autoplaced yes)
 		(property "Reference" "#PWR017"
-			(at 166.37 128.27 0)
+			(at 252.73 86.36 0)
 			(effects
 				(font
@@
 			)
 		)
-		(property "Value" "VBUS"
-			(at 166.37 119.38 0)
+		(property "Value" "+3V3"
+			(at 252.73 77.47 0)
 			(effects
 				(font
@@
 		)
 		(property "Footprint" ""
-			(at 166.37 124.46 0)
+			(at 252.73 82.55 0)
 			(effects
 				(font
@@
 		)
 		(property "Datasheet" ""
-			(at 166.37 124.46 0)
+			(at 252.73 82.55 0)
 			(effects
 				(font
@@
 			)
 		)
-		(property "Description" "Power symbol creates a global label with name \"VBUS\""
-			(at 166.37 124.46 0)
+		(property "Description" "Power symbol creates a global label with name \"+3V3\""
+			(at 252.73 82.55 0)
 			(effects
 				(font

Commit message: bom done
Other:
- note removed: "55V MAX!"
Changed lines of the file:
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@@
 		(comment 2 "Designed in poland")
-	)
-	(text "55V MAX!"
-		(exclude_from_sim no)
-		(at 54.864 172.212 0)
-		(effects
-			(font
-				(size 5.08 5.08)
-				(thickness 10.16)
-				(bold yes)
-			)
-		)
 	)
 	(junction

Commit message: REV A production ready
Connections:
- no-connect marks 0 -> 1
Changed lines of the file:
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@@
 		(color 0 0 0 0)
+	)
+	(no_connect
+		(at 110.49 95.25)
 	)
 	(wire
@@
 		)
 		(stroke
+			(width 0)
+			(type default)
+		)
+	)
+	(wire
+		(pts
+			(xy 104.14 95.25) (xy 110.49 95.25)
+		)
+		(stroke
